Commit message: first commit

File: magni_description/urdf/inertial.xacro (robot description, xacro)
@@ -25,5 +25,5 @@
 -->
 <robot xmlns:xacro="http://wiki.ros.org/xacro">
-    <property name="M_PI" value="3.1415926535897931" />
+    <xacro:property name="M_PI" value="3.1415926535897931" />
     <!-- see https://secure.wikimedia.org/wikipedia/en/wiki/List_of_moment_of_inertia_tensors -->
     <!-- #################### versions without origin #################### -->
@@ -59,5 +59,5 @@
         <inertial>
             <mass value="${mass}" />
-            <insert_block name="origin" />
+            <xacro:insert_block name="origin" />
             <inertia ixx="${0.4 * mass * radius * radius}" ixy="0.0" ixz="0.0"
                      iyy="${0.4 * mass * radius * radius}" iyz="0.0"
@@ -68,5 +68,5 @@
         <inertial>
             <mass value="${mass}" />
-            <insert_block name="origin" />
+            <xacro:insert_block name="origin" />
             <inertia ixx="${0.0833333 * mass * (3 * radius * radius + length * length)}" ixy="0.0" ixz="0.0"
                      iyy="${0.0833333 * mass * (3 * radius * radius + length * length)}" iyz="0.0"
@@ -77,5 +77,5 @@
         <inertial>
             <mass value="${mass}" />
-            <insert_block name="origin" />
+            <xacro:insert_block name="origin" />
             <inertia ixx="${0.0833333 * mass * (y*y + z*z)}" ixy="0.0" ixz="0.0"
                      iyy="${0.0833333 * mass * (x*x + z*z)}" iyz="0.0"

File: magni_description/urdf/magni.urdf.xacro (robot description, xacro)
@@ -1,4 +1,8 @@
 <?xml version="1.0"?>
 <robot xmlns:xacro="http://wiki.ros.org/xacro" name="magni">
+  <xacro:arg name="laser_enabled" default="true" />
+  <xacro:property name="laser_enabled" value="$(arg laser_enabled)"/>
+  <xacro:property name="laser_xyz" default="0.2206 0.0 0.00635" />
+  <xacro:property name="laser_rpy" default="0.0 0.0 0.0)" />
   <xacro:arg name="raspicam_mount" default="forward"/>
   <xacro:property name="raspicam_mount" value="$(arg raspicam_mount)"/>
@@ -14,4 +18,5 @@
   <xacro:include filename="$(find magni_description)/urdf/sensors/sonar_hc-sr04.xacro" />
   <xacro:include filename="$(find magni_description)/urdf/sensors/raspi_camera.xacro" />
+  <xacro:include filename="$(find hector_sensors_description)/urdf/hokuyo_utm30lx.urdf.xacro"/>
   <!-- Robot base_link -->
   <link name="base_link">
@@ -138,4 +143,9 @@
     </xacro:sonar_hc-sr04>
   </xacro:if>
+  <xacro:if value="${laser_enabled}">
+    <xacro:hokuyo_utm30lx name="hokuyo_laser" parent="base_link" ros_topic="scan" update_rate="10" ray_count="361" min_angle="-180" max_angle="180">
+      <origin xyz="0 0 +0.25" rpy="0 0 0" />
+    </xacro:hokuyo_utm30lx>
+  </xacro:if>
   <!-- If we are given an extrinsics calibration use that instead of the pre-configured pose -->
   <xacro:if value="${camera_extrinsics_file != '-'}">
