Commit message: added realsense camera

File: magni_description/urdf/magni.urdf.xacro (robot description, xacro)
@@ -93,5 +93,5 @@
     </inertial>
   </link>
-  <joint name="camera_joint" type="fixed">
+  <joint name="camera_RGB_joint" type="fixed">
     <axis xyz="0 1 0" />
     <origin xyz="0 0 1.5" rpy="0 0 0"/>
@@ -99,5 +99,9 @@
     <child link="camera"/>
   </joint>
-  <!-- RGB camera, might use RGBD camera -->
+  <!-- realsense camera -->
+ <xacro:include filename="$(find magni_description)/urdf/_d435.urdf.xacro" />
+  <xacro:sensor_d435  parent="base_link">
+    <origin xyz="0.0 0 1.3" rpy="0 0 0"/>
+  </xacro:sensor_d435>
   <!-- Fixed offset from the floor to the center of the wheels -->
   <link name="base_footprint"/>
