Commit message: modify topics to match with spencer package

File: magni_description/urdf/_d435.gazebo.xacro (robot description, xacro)
@@ -43,5 +43,5 @@
         <always_on>1</always_on>
         <update_rate>30</update_rate>
-        <visualize>1</visualize>
+        <visualize>0</visualize>
       </sensor>
       <sensor name="${camera_name}ired1" type="camera">
@@ -49,6 +49,6 @@
           <horizontal_fov>${85.2*deg_to_rad}</horizontal_fov>
           <image>
-            <width>1280</width>
-            <height>720</height>
+            <width>640</width>
+            <height>480</height>
             <format>L_INT8</format>
           </image>
@@ -71,6 +71,6 @@
           <horizontal_fov>${85.2*deg_to_rad}</horizontal_fov>
           <image>
-            <width>1280</width>
-            <height>720</height>
+            <width>640</width>
+            <height>480</height>
             <format>L_INT8</format>
           </image>
@@ -93,6 +93,6 @@
           <horizontal_fov>${85.2*deg_to_rad}</horizontal_fov>
           <image>
-            <width>1280</width>
-            <height>720</height>
+            <width>640</width>
+            <height>480</height>
           </image>
           <clip>
@@ -117,8 +117,8 @@
         <colorUpdateRate>30.0</colorUpdateRate>
         <infraredUpdateRate>30.0</infraredUpdateRate>
-        <depthTopicName>depth/image_raw</depthTopicName>
+        <depthTopicName>depth/image_rect_raw</depthTopicName>
         <depthCameraInfoTopicName>depth/camera_info</depthCameraInfoTopicName>
-        <colorTopicName>color/image_raw</colorTopicName>
-        <colorCameraInfoTopicName>color/camera_info</colorCameraInfoTopicName>
+        <colorTopicName>rgb/image_rect_color</colorTopicName>
+        <colorCameraInfoTopicName>rgb/camera_info</colorCameraInfoTopicName>
         <infrared1TopicName>infra1/image_raw</infrared1TopicName>
         <infrared1CameraInfoTopicName>infra1/camera_info</infrared1CameraInfoTopicName>

File: magni_description/urdf/magni.gazebo.xacro (robot description, xacro)
@@ -40,36 +40,3 @@
         <kp>1e8</kp>
     </gazebo>
-    <!-- RGB camera, might use RGBD camera -->
-    <gazebo reference="camera">
-        <material>Gazebo/Green</material>
-        <sensor type="camera" name="RGBD_camera">
-            <update_rate>30.0</update_rate>
-            <camera name="head">
-                <horizontal_fov>1.3962634</horizontal_fov>
-                <image>
-                    <width>1600</width>
-                    <height>1600</height>
-                    <format>R8G8B8</format>
-                </image>
-                <clip>
-                    <near>0.02</near>
-                    <far>300</far>
-                </clip>
-            </camera>
-            <plugin name="camera_controller" filename="libgazebo_ros_camera.so">
-                <alwaysOn>true</alwaysOn>
-                <updateRate>0.0</updateRate>
-                <cameraName>magni/RGBD_camera</cameraName>
-                <imageTopicName>image_raw</imageTopicName>
-                <cameraInfoTopicName>camera_info</cameraInfoTopicName>
-                <frameName>camera</frameName>
-                <hackBaseline>0.07</hackBaseline>
-                <distortionK1>0.0</distortionK1>
-                <distortionK2>0.0</distortionK2>
-                <distortionK3>0.0</distortionK3>
-                <distortionT1>0.0</distortionT1>
-                <distortionT2>0.0</distortionT2>
-            </plugin>
-        </sensor>
-    </gazebo>
 </robot>

File: magni_description/urdf/magni.urdf.xacro (robot description, xacro)
@@ -20,6 +20,19 @@
   <xacro:include filename="$(find magni_description)/urdf/sensors/sonar_hc-sr04.xacro" />
   <xacro:include filename="$(find magni_description)/urdf/sensors/raspi_camera.xacro" />
-  <xacro:include filename="$(find hector_sensors_description)/urdf/hokuyo_utm30lx.urdf.xacro"/>
-  <!-- <xacro:include filename="$(find magni_description)/urdf/_d435.urdf.xacro"/> -->
+  <xacro:include filename="$(find magni_description)/urdf/hokuyo_utm30lx.urdf.xacro"/>
+  <xacro:include filename="$(find magni_description)/urdf/_d435.urdf.xacro"/>
+  <link name="rod_camera2base">
+    <visual>
+      <origin xyz="0 0 0.25" rpy="0 0 0" />
+      <geometry>
+        <cylinder radius="0.013" length="1.2"/>
+      </geometry>
+    </visual>
+  </link>
+  <joint name="rod_camera2base_joint" type="fixed">
+    <parent link="base_link"/>
+    <child link="rod_camera2base"/>
+    <origin xyz="-0.05 0 0.512" rpy="0 0 0"/>
+  </joint>
   <!-- Robot base_link -->
   <link name="base_link">
@@ -30,5 +43,5 @@
       </geometry>
     </visual>
-	<visual>
+    <visual>
       <origin xyz="${-wheel_xpos-0.169} 0.17 ${-wheel_r+0.09}" rpy="0 0 ${pi}" />
       <geometry>
@@ -36,5 +49,5 @@
       </geometry>
     </visual>
-	<visual>
+    <visual>
       <origin xyz="${-wheel_xpos-0.169} -0.17 ${-wheel_r+0.09}" rpy="0 0 ${pi}" />
       <geometry>
@@ -43,5 +56,5 @@
     </visual>
     <collision>
-	  <origin xyz="${-wheel_xpos} 0 ${-wheel_r+0.151}" rpy="0 0 0" />
+      <origin xyz="${-wheel_xpos} 0 ${-wheel_r+0.151}" rpy="0 0 0" />
       <geometry>
         <box size="0.398 0.268 0.160"/>
@@ -66,41 +79,12 @@
       </geometry>
     </collision>
-    <xacro:box_inertial_with_origin  x="0.398" y="0.221" z="0.150" mass="10.0">
+    <xacro:box_inertial_with_origin x="0.398" y="0.221" z="0.150" mass="10.0">
       <origin xyz="-0.15 0 0.03" rpy="0 0 0" />
     </xacro:box_inertial_with_origin>
   </link>
-  <!-- RGB camera, might use RGBD camera -->
-  <link name="camera">
-    <collision>
-      <origin xyz="0 0 0" rpy="0 0 0"/>
-      <geometry>
-        <box size="${cameraSize} ${cameraSize} ${cameraSize}"/>
-      </geometry>
-    </collision>
-    <visual>
-      <origin xyz="0 0 0" rpy="0 0 0"/>
-      <geometry>
-        <box size="${cameraSize} ${cameraSize} ${cameraSize}"/>
-        <!-- <mesh filename="package://magni_description/meshes/d435.dae" /> -->
-      </geometry>
-      <!-- <material name="green"/> -->
-    </visual>
-    <inertial>
-      <mass value="${cameraMass}" />
-      <origin xyz="0 0 0" rpy="0 0 0"/>
-      <box_inertia m="${cameraMass}" x="${cameraSize}" y="${cameraSize}" z="${cameraSize}" />
-      <inertia ixx="1e-6" ixy="0" ixz="0" iyy="1e-6" iyz="0" izz="1e-6" />
-    </inertial>
-  </link>
-  <joint name="camera_RGB_joint" type="fixed">
-    <axis xyz="0 1 0" />
-    <origin xyz="0 0 1.5" rpy="0 0 0"/>
-    <parent link="base_link"/>
-    <child link="camera"/>
-  </joint>
   <!-- realsense camera -->
- <xacro:include filename="$(find magni_description)/urdf/_d435.urdf.xacro" />
-  <xacro:sensor_d435  parent="base_link">
-    <origin xyz="0.0 0 1.3" rpy="0 0 0"/>
+  <xacro:include filename="$(find magni_description)/urdf/_d435.urdf.xacro" />
+  <xacro:sensor_d435 parent="base_link">
+    <origin xyz="-0.0256 0 1.3" rpy="0 0 0"/>
   </xacro:sensor_d435>
   <!-- Fixed offset from the floor to the center of the wheels -->
@@ -191,6 +175,5 @@
     <xacro:property name="cam_orientation" value="${cam_extrinsics['orientation']}"/>
     <xacro:raspi_camera name="raspicam" connected_to="base_link">
-      <origin xyz="${cam_position['x']} ${cam_position['y']} ${cam_position['z']}"
-        rpy="${cam_orientation['r']} ${cam_orientation['p']} ${cam_orientation['y']}"/>
+      <origin xyz="${cam_position['x']} ${cam_position['y']} ${cam_position['z']}" rpy="${cam_orientation['r']} ${cam_orientation['p']} ${cam_orientation['y']}"/>
     </xacro:raspi_camera>
   </xacro:if>
