Commit message: remove achieve, restructure file and add velodyne 3D lidar plugin into the magni model

File: magni_description/urdf/_d435.urdf.xacro (robot description, xacro)
@@ -49,5 +49,5 @@
           <!-- <box size="${d435_cam_width} ${d435_cam_height} ${d435_cam_depth}"/> -->
           <mesh filename="package://magni_description/meshes/d435.dae" />
-          <!--<mesh filename="package://realsense2_description/meshes/d435/d435.dae" />-->
+          <!-- <mesh filename="package://realsense2_description/meshes/d435/d435.dae" /> -->
         </geometry>
         <material name="${name}_aluminum"/>

File: magni_description/urdf/magni.urdf.xacro (robot description, xacro)
@@ -1,6 +1,6 @@
 <?xml version="1.0"?>
 <robot xmlns:xacro="http://wiki.ros.org/xacro" name="magni">
-  <xacro:arg name="laser_enabled" default="true" />
-  <xacro:property name="laser_enabled" value="$(arg laser_enabled)"/>
+  <xacro:arg name="hokuyo_laser_enabled" default="true" />
+  <xacro:property name="hokuyo_laser_enabled" value="$(arg hokuyo_laser_enabled)"/>
   <xacro:property name="laser_xyz" default="0.2206 0.0 0.00635" />
   <xacro:property name="laser_rpy" default="0.0 0.0 0.0)" />
@@ -15,4 +15,10 @@
   <xacro:property name="wheel_r" value="0.1" />
   <xacro:property name="wheel_xpos" value="0.11" />
+  <xacro:arg name="realsense_camera_enabled" default="false" />
+  <xacro:property name="realsense_camera_enabled" value="$(arg realsense_camera_enabled)"/>
+  <xacro:arg name="velodyne_laser_enabled" default="false" />
+  <xacro:property name="velodyne_laser_enabled" value="$(arg velodyne_laser_enabled)"/>
+  <xacro:arg name="gpu" default="true"/>
+  <xacro:property name="gpu" value="$(arg gpu)" />
   <xacro:include filename="$(find magni_description)/urdf/magni.transmission.xacro" />
   <xacro:include filename="$(find magni_description)/urdf/magni.gazebo.xacro" />
@@ -22,17 +28,24 @@
   <xacro:include filename="$(find magni_description)/urdf/hokuyo_utm30lx.urdf.xacro"/>
   <xacro:include filename="$(find magni_description)/urdf/_d435.urdf.xacro"/>
-  <link name="rod_camera2base">
-    <visual>
-      <origin xyz="0 0 0.25" rpy="0 0 0" />
-      <geometry>
-        <cylinder radius="0.013" length="1.2"/>
-      </geometry>
-    </visual>
-  </link>
-  <joint name="rod_camera2base_joint" type="fixed">
-    <parent link="base_link"/>
-    <child link="rod_camera2base"/>
-    <origin xyz="-0.05 0 0.512" rpy="0 0 0"/>
-  </joint>
+  <xacro:if value="${realsense_camera_enabled}">
+    <link name="rod_camera2base">
+      <visual>
+        <origin xyz="0 0 0.25" rpy="0 0 0" />
+        <geometry>
+          <cylinder radius="0.013" length="1.2"/>
+        </geometry>
+      </visual>
+    </link>
+    <!-- realsense camera -->
+    <xacro:include filename="$(find magni_description)/urdf/_d435.urdf.xacro" />
+    <xacro:sensor_d435 parent="base_link">
+      <origin xyz="-0.2256 0 1.3" rpy="0 0 0"/>
+    </xacro:sensor_d435>
+    <joint name="rod_camera2base_joint" type="fixed">
+      <parent link="base_link"/>
+      <child link="rod_camera2base"/>
+      <origin xyz="-0.25 0 0.512" rpy="0 0 0"/>
+    </joint>
+  </xacro:if>
   <!-- Robot base_link -->
   <link name="base_link">
@@ -83,9 +96,4 @@
     </xacro:box_inertial_with_origin>
   </link>
-  <!-- realsense camera -->
-  <xacro:include filename="$(find magni_description)/urdf/_d435.urdf.xacro" />
-  <xacro:sensor_d435 parent="base_link">
-    <origin xyz="-0.0256 0 1.3" rpy="0 0 0"/>
-  </xacro:sensor_d435>
   <!-- Fixed offset from the floor to the center of the wheels -->
   <link name="base_footprint"/>
@@ -164,5 +172,5 @@
     </xacro:sonar_hc-sr04>
   </xacro:if>
-  <xacro:if value="${laser_enabled}">
+  <xacro:if value="${hokuyo_laser_enabled}">
     <xacro:hokuyo_utm30lx name="hokuyo_laser" parent="base_link" ros_topic="scan" update_rate="10" ray_count="361" min_angle="-180" max_angle="180">
       <origin xyz="0 0 +0.25" rpy="0 0 0" />
@@ -205,3 +213,10 @@
     </xacro:if>
   </xacro:if>
+  <xacro:if value="${velodyne_laser_enabled}">
+    <!-- VLP-16 -->
+    <xacro:include filename="$(find velodyne_description)/urdf/VLP-16.urdf.xacro"/>
+    <xacro:VLP-16 parent="base_link" name="velodyne" topic="/velodyne_points" organize_cloud="false" hz="10" samples="440" gpu="${gpu}">
+      <origin xyz="-0.1 0 0.4" rpy="0 0 0" />
+    </xacro:VLP-16>
+  </xacro:if>
 </robot>

Commit message: namespaced tf_prefix, topic_ns and node_ns

File: magni_description/urdf/_d435.urdf.xacro (robot description, xacro)
@@ -8,7 +8,7 @@
 <robot name="sensor_d435" xmlns:xacro="http://ros.org/wiki/xacro">
   <!--File includes-->
-  <xacro:include filename="$(find magni_description)/urdf/_d435.gazebo.xacro"/>
-  <xacro:macro name="sensor_d435" params="name:=camera topics_ns:=camera parent *origin publish_pointcloud:=true">
+  <xacro:macro name="sensor_d435" params="name:=camera topics_ns:=camera tf_prefix parent *origin publish_pointcloud:=true">
     <xacro:property name="M_PI" value="3.1415926535897931" />
+    <xacro:include filename="$(find magni_description)/urdf/_d435.gazebo.xacro"/>
     <!-- The following values are approximate, and the camera node
      publishing TF values with actual calibrated camera extrinsic values -->
@@ -28,20 +28,20 @@
     <xacro:property name="d435_cam_depth_py" value="0.0175"/>
     <xacro:property name="d435_cam_depth_pz" value="${d435_cam_height/2}"/>
-    <material name="${name}_aluminum">
+    <material name="${tf_prefix}${name}_aluminum">
     <color rgba="0.5 0.5 0.5 1"/>
     </material>
     <!-- camera body, with origin at bottom screw mount -->
-    <joint name="${name}_joint" type="fixed">
+    <joint name="${tf_prefix}${name}_joint" type="fixed">
       <xacro:insert_block name="origin" />
       <parent link="${parent}"/>
-      <child link="${name}_bottom_screw_frame" />
+      <child link="${tf_prefix}${name}_bottom_screw_frame" />
     </joint>
-    <link name="${name}_bottom_screw_frame"/>
-    <joint name="${name}_link_joint" type="fixed">
+    <link name="${tf_prefix}${name}_bottom_screw_frame"/>
+    <joint name="${tf_prefix}${name}_link_joint" type="fixed">
       <origin xyz="0 ${d435_cam_depth_py} ${d435_cam_depth_pz}" rpy="0 0 0"/>
-      <parent link="${name}_bottom_screw_frame"/>
-      <child link="${name}_link" />
+      <parent link="${tf_prefix}${name}_bottom_screw_frame"/>
+      <child link="${tf_prefix}${name}_link" />
     </joint>
-    <link name="${name}_link">
+    <link name="${tf_prefix}${name}_link">
       <visual>
       <origin xyz="${d435_cam_mount_from_center_offset} ${-d435_cam_depth_py} 0" rpy="${M_PI/2} 0 ${M_PI/2}"/>
@@ -51,5 +51,5 @@
           <!--<mesh filename="package://realsense2_description/meshes/d435/d435.dae" />-->
         </geometry>
-        <material name="${name}_aluminum"/>
+        <material name="${tf_prefix}${name}_aluminum"/>
       </visual>
       <collision>
@@ -67,57 +67,57 @@
     </link>
     <!-- camera depth joints and links -->
-    <joint name="${name}_depth_joint" type="fixed">
+    <joint name="${tf_prefix}${name}_depth_joint" type="fixed">
       <origin xyz="0 0 0" rpy="0 0 0"/>
-      <parent link="${name}_link"/>
-      <child link="${name}_depth_frame" />
+      <parent link="${tf_prefix}${name}_link"/>
+      <child link="${tf_prefix}${name}_depth_frame" />
     </joint>
-    <link name="${name}_depth_frame"/>
-    <joint name="${name}_depth_optical_joint" type="fixed">
+    <link name="${tf_prefix}${name}_depth_frame"/>
+    <joint name="${tf_prefix}${name}_depth_optical_joint" type="fixed">
       <origin xyz="0 0 0" rpy="${-M_PI/2} 0 ${-M_PI/2}" />
-      <parent link="${name}_depth_frame" />
-      <child link="${name}_depth_optical_frame" />
+      <parent link="${tf_prefix}${name}_depth_frame" />
+      <child link="${tf_prefix}${name}_depth_optical_frame" />
     </joint>
-    <link name="${name}_depth_optical_frame"/>
+    <link name="${tf_prefix}${name}_depth_optical_frame"/>
     <!-- camera left IR joints and links -->
-    <joint name="${name}_left_ir_joint" type="fixed">
+    <joint name="${tf_prefix}${name}_left_ir_joint" type="fixed">
       <origin xyz="0 ${d435_cam_depth_to_left_ir_offset} 0" rpy="0 0 0" />
-      <parent link="${name}_depth_frame" />
-      <child link="${name}_left_ir_frame" />
+      <parent link="${tf_prefix}${name}_depth_frame" />
+      <child link="${tf_prefix}${name}_left_ir_frame" />
     </joint>
-    <link name="${name}_left_ir_frame"/>
-    <joint name="${name}_left_ir_optical_joint" type="fixed">
+    <link name="${tf_prefix}${name}_left_ir_frame"/>
+    <joint name="${tf_prefix}${name}_left_ir_optical_joint" type="fixed">
       <origin xyz="0 0 0" rpy="${-M_PI/2} 0 ${-M_PI/2}" />
-      <parent link="${name}_left_ir_frame" />
-      <child link="${name}_left_ir_optical_frame" />
+      <parent link="${tf_prefix}${name}_left_ir_frame" />
+      <child link="${tf_prefix}${name}_left_ir_optical_frame" />
     </joint>
-    <link name="${name}_left_ir_optical_frame"/>
+    <link name="${tf_prefix}${name}_left_ir_optical_frame"/>
     <!-- camera right IR joints and links -->
-    <joint name="${name}_right_ir_joint" type="fixed">
+    <joint name="${tf_prefix}${name}_right_ir_joint" type="fixed">
       <origin xyz="0 ${d435_cam_depth_to_right_ir_offset} 0" rpy="0 0 0" />
-      <parent link="${name}_depth_frame" />
-      <child link="${name}_right_ir_frame" />
+      <parent link="${tf_prefix}${name}_depth_frame" />
+      <child link="${tf_prefix}${name}_right_ir_frame" />
     </joint>
-    <link name="${name}_right_ir_frame"/>
-    <joint name="${name}_right_ir_optical_joint" type="fixed">
+    <link name="${tf_prefix}${name}_right_ir_frame"/>
+    <joint name="${tf_prefix}${name}_right_ir_optical_joint" type="fixed">
       <origin xyz="0 0 0" rpy="${-M_PI/2} 0 ${-M_PI/2}" />
-      <parent link="${name}_right_ir_frame" />
-      <child link="${name}_right_ir_optical_frame" />
+      <parent link="${tf_prefix}${name}_right_ir_frame" />
+      <child link="${tf_prefix}${name}_right_ir_optical_frame" />
     </joint>
-    <link name="${name}_right_ir_optical_frame"/>
+    <link name="${tf_prefix}${name}_right_ir_optical_frame"/>
     <!-- camera color joints and links -->
-    <joint name="${name}_color_joint" type="fixed">
+    <joint name="${tf_prefix}${name}_color_joint" type="fixed">
       <origin xyz="0 ${d435_cam_depth_to_color_offset} 0" rpy="0 0 0" />
-      <parent link="${name}_depth_frame" />
-      <child link="${name}_color_frame" />
+      <parent link="${tf_prefix}${name}_depth_frame" />
+      <child link="${tf_prefix}${name}_color_frame" />
     </joint>
-    <link name="${name}_color_frame"/>
-    <joint name="${name}_color_optical_joint" type="fixed">
+    <link name="${tf_prefix}${name}_color_frame"/>
+    <joint name="${tf_prefix}${name}_color_optical_joint" type="fixed">
       <origin xyz="0 0 0" rpy="${-M_PI/2} 0 ${-M_PI/2}" />
-      <parent link="${name}_color_frame" />
-      <child link="${name}_color_optical_frame" />
+      <parent link="${tf_prefix}${name}_color_frame" />
+      <child link="${tf_prefix}${name}_color_optical_frame" />
     </joint>
-    <link name="${name}_color_optical_frame"/>
+    <link name="${tf_prefix}${name}_color_optical_frame"/>
     <!-- Realsense Gazebo Plugin -->
-    <xacro:gazebo_d435 camera_name="${name}" reference_link="${name}_link" topics_ns="${topics_ns}" depth_optical_frame="${name}_depth_optical_frame" color_optical_frame="${name}_color_optical_frame" infrared1_optical_frame="${name}_left_ir_optical_frame" infrared2_optical_frame="${name}_right_ir_optical_frame" publish_pointcloud="${publish_pointcloud}"/>
+    <xacro:gazebo_d435 camera_name="${tf_prefix}${name}" reference_link="${tf_prefix}${name}_link" topics_ns="${tf_prefix}" depth_optical_frame="${tf_prefix}${name}_depth_optical_frame" color_optical_frame="${tf_prefix}${name}_color_optical_frame" infrared1_optical_frame="${tf_prefix}${name}_left_ir_optical_frame" infrared2_optical_frame="${tf_prefix}${name}_right_ir_optical_frame" publish_pointcloud="${publish_pointcloud}"/>
   </xacro:macro>
 </robot>

File: magni_description/urdf/magni.gazebo.xacro (robot description, xacro)
@@ -1,7 +1,7 @@
 <?xml version="1.0"?>
 <robot xmlns:xacro="http://wiki.ros.org/xacro">
+     <xacro:arg name="tf_prefix" default="" />
     <gazebo>
         <plugin name="gazebo_ros_control" filename="libgazebo_ros_control.so">
-            <legacyModeNS>true</legacyModeNS>
         </plugin>
     </gazebo>
@@ -9,5 +9,5 @@
         <plugin name="gazebo_ros_p3d" filename="libgazebo_ros_p3d.so">
             <updateRate>100</updateRate>
-            <bodyName>base_footprint</bodyName>
+            <bodyName>${tf_prefix}base_footprint</bodyName>
             <topicName>exact_pose</topicName>
             <frameName>map</frameName>

File: magni_description/urdf/magni.transmission.xacro (robot description, xacro)
@@ -1,20 +1,20 @@
 <?xml version="1.0"?>
 <robot xmlns:xacro="http://wiki.ros.org/xacro">
-    <transmission name="left_wheel_transmission">
+    <transmission name="${tf_prefix}left_wheel_transmission">
         <type>transmission_interface/SimpleTransmission</type>
-        <joint name="left_wheel_joint">
+        <joint name="${tf_prefix}left_wheel_joint">
             <hardwareInterface>hardware_interface/VelocityJointInterface</hardwareInterface>
         </joint>
-        <actuator name="left_wheel_actuator">
+        <actuator name="${tf_prefix}left_wheel_actuator">
             <mechanicalReduction>1</mechanicalReduction>
             <hardwareInterface>VelocityJointInterface</hardwareInterface>
         </actuator>
     </transmission>
-    <transmission name="right_wheel_transmission">
+    <transmission name="${tf_prefix}right_wheel_transmission">
         <type>transmission_interface/SimpleTransmission</type>
-        <joint name="right_wheel_joint">
+        <joint name="${tf_prefix}right_wheel_joint">
             <hardwareInterface>hardware_interface/VelocityJointInterface</hardwareInterface>
         </joint>
-        <actuator name="right_wheel_actuator">
+        <actuator name="${tf_prefix}right_wheel_actuator">
             <mechanicalReduction>1</mechanicalReduction>
             <hardwareInterface>VelocityJointInterface</hardwareInterface>

File: magni_description/urdf/magni.urdf.xacro (robot description, xacro)
@@ -2,4 +2,6 @@
 <robot xmlns:xacro="http://wiki.ros.org/xacro" name="magni">
   <xacro:arg name="laser_enabled" default="true" />
+  <xacro:arg name="tf_prefix" default="" />
+  <xacro:property name="tf_prefix" value="$(arg tf_prefix)" />
   <xacro:property name="laser_enabled" value="$(arg laser_enabled)"/>
   <xacro:property name="laser_xyz" default="0.2206 0.0 0.00635" />
@@ -22,5 +24,5 @@
   <xacro:include filename="$(find magni_description)/urdf/hokuyo_utm30lx.urdf.xacro"/>
   <xacro:include filename="$(find magni_description)/urdf/_d435.urdf.xacro"/>
-  <link name="rod_camera2base">
+  <link name="${tf_prefix}rod_camera2base">
     <visual>
       <origin xyz="0 0 0.25" rpy="0 0 0" />
@@ -30,11 +32,11 @@
     </visual>
   </link>
-  <joint name="rod_camera2base_joint" type="fixed">
-    <parent link="base_link"/>
-    <child link="rod_camera2base"/>
+  <joint name="${tf_prefix}brod_camera2base_joint" type="fixed">
+    <parent link="${tf_prefix}base_link"/>
+    <child link="${tf_prefix}rod_camera2base"/>
     <origin xyz="-0.05 0 0.512" rpy="0 0 0"/>
   </joint>
   <!-- Robot base_link -->
-  <link name="base_link">
+  <link name="${tf_prefix}base_link">
     <visual>
       <origin xyz="${-wheel_xpos} 0 ${-wheel_r+0.071}" rpy="0 0 0" />
@@ -85,17 +87,17 @@
   <!-- realsense camera -->
   <xacro:include filename="$(find magni_description)/urdf/_d435.urdf.xacro" />
-  <xacro:sensor_d435 parent="base_link">
+  <xacro:sensor_d435 parent="${tf_prefix}base_link" tf_prefix="${tf_prefix}">
     <origin xyz="-0.0256 0 1.3" rpy="0 0 0"/>
   </xacro:sensor_d435>
   <!-- Fixed offset from the floor to the center of the wheels -->
-  <link name="base_footprint"/>
-  <joint name="base_footprint_joint" type="fixed">
-    <parent link="base_footprint"/>
-    <child link="base_link"/>
+  <link name="${tf_prefix}base_footprint"/>
+  <joint name="${tf_prefix}bbase_footprint_joint" type="fixed">
+    <parent link="${tf_prefix}base_footprint"/>
+    <child link="${tf_prefix}base_link"/>
     <origin xyz="0 0 ${wheel_r}" rpy="0 0 0"/>
   </joint>
   <!-- Macro for defining wheels -->
   <xacro:macro name="wheel" params="prefix reflect">
-    <link name="${prefix}_wheel">
+    <link name="${tf_prefix}${prefix}_wheel">
       <visual>
         <origin xyz="${-0.071*reflect} 0 0" rpy="0 ${(reflect-1)*pi/2} 0" />
@@ -120,8 +122,8 @@
       </xacro:cylinder_inertial_with_origin>
     </link>
-    <joint name="${prefix}_wheel_joint" type="continuous">
+    <joint name="${tf_prefix}${prefix}_wheel_joint" type="continuous">
       <axis xyz="1 0 0" rpy="0 0 0" />
-      <parent link="base_link"/>
-      <child link="${prefix}_wheel"/>
+      <parent link="${tf_prefix}base_link"/>
+      <child link="${tf_prefix}${prefix}_wheel"/>
       <origin xyz="0 ${0.163*reflect} 0" rpy="0 0 ${pi/2}"/>
     </joint>
@@ -131,5 +133,5 @@
   <!-- Macro for defining caster wheels -->
   <xacro:macro name="caster_wheel" params="prefix reflect">
-    <link name="${prefix}_caster_wheel">
+    <link name="${tf_prefix}${prefix}_caster_wheel">
       <collision>
         <origin xyz="${-wheel_xpos-0.19} ${reflect*0.169} ${-wheel_r+0.04}" rpy="0 0 0" />
@@ -139,7 +141,7 @@
       </collision>
     </link>
-    <joint name="${prefix}_caster_wheel_joint" type="fixed">
-      <parent link="base_link"/>
-      <child link="${prefix}_caster_wheel"/>
+    <joint name="${tf_prefix}b${prefix}_caster_wheel_joint" type="fixed">
+      <parent link="${tf_prefix}base_link"/>
+      <child link="${tf_prefix}${prefix}_caster_wheel"/>
     </joint>
   </xacro:macro>
@@ -148,22 +150,22 @@
   <!-- Define all sonars, if sonars_installed set to 1 -->
   <xacro:if value="${sonars_installed}">
-    <xacro:sonar_hc-sr04 name="sonar_0" connected_to="base_link">
+    <xacro:sonar_hc-sr04 name="sonar_0" connected_to="${tf_prefix}base_link">
       <origin xyz="0.01 -0.14 0.15" rpy="0 0 ${-pi/2}"/>
     </xacro:sonar_hc-sr04>
-    <xacro:sonar_hc-sr04 name="sonar_1" connected_to="base_link">
+    <xacro:sonar_hc-sr04 name="sonar_1" connected_to="${tf_prefix}base_link">
       <origin xyz="0.08 -0.07 0.15" rpy="0 0 0.785"/>
     </xacro:sonar_hc-sr04>
-    <xacro:sonar_hc-sr04 name="sonar_2" connected_to="base_link">
+    <xacro:sonar_hc-sr04 name="sonar_2" connected_to="${tf_prefix}base_link">
       <origin xyz="0.08 -0.01 0.15" rpy="0 0 -0.785"/>
     </xacro:sonar_hc-sr04>
-    <xacro:sonar_hc-sr04 name="sonar_3" connected_to="base_link">
+    <xacro:sonar_hc-sr04 name="sonar_3" connected_to="${tf_prefix}base_link">
       <origin xyz="0.08 0.04 0.15" rpy="0 0 0"/>
     </xacro:sonar_hc-sr04>
-    <xacro:sonar_hc-sr04 name="sonar_4" connected_to="base_link">
+    <xacro:sonar_hc-sr04 name="sonar_4" connected_to="${tf_prefix}base_link">
       <origin xyz="0.01 0.14 0.15" rpy="0 0 ${pi/2}"/>
     </xacro:sonar_hc-sr04>
   </xacro:if>
   <xacro:if value="${laser_enabled}">
-    <xacro:hokuyo_utm30lx name="hokuyo_laser" parent="base_link" ros_topic="scan" update_rate="10" ray_count="361" min_angle="-180" max_angle="180">
+    <xacro:hokuyo_utm30lx name="${tf_prefix}hokuyo_laser" parent="${tf_prefix}base_link" ros_topic="${tf_prefix}scan" update_rate="10" ray_count="361" min_angle="-180" max_angle="180">
       <origin xyz="0 0 +0.25" rpy="0 0 0" />
     </xacro:hokuyo_utm30lx>
@@ -174,5 +176,5 @@
     <xacro:property name="cam_position" value="${cam_extrinsics['position']}"/>
     <xacro:property name="cam_orientation" value="${cam_extrinsics['orientation']}"/>
-    <xacro:raspi_camera name="raspicam" connected_to="base_link">
+    <xacro:raspi_camera name="${tf_prefix}raspicam" connected_to="${tf_prefix}base_link">
       <origin xyz="${cam_position['x']} ${cam_position['y']} ${cam_position['z']}" rpy="${cam_orientation['r']} ${cam_orientation['p']} ${cam_orientation['y']}"/>
     </xacro:raspi_camera>
@@ -185,20 +187,20 @@
     <!-- ahead    Directly facing forward with no tilt        -->
     <xacro:if value="${raspicam_mount == 'forward'}">
-      <xacro:raspi_camera name="raspicam" connected_to="base_link">
+      <xacro:raspi_camera name="${tf_prefix}raspicam" connected_to="${tf_prefix}base_link">
         <origin xyz="0.050 0.085 0.135" rpy="1.15191731 0 1.5707"/>
       </xacro:raspi_camera>
     </xacro:if>
     <xacro:if value="${raspicam_mount == 'upward'}">
-      <xacro:raspi_camera name="raspicam" connected_to="base_link">
+      <xacro:raspi_camera name="${tf_prefix}raspicam" connected_to="${tf_prefix}base_link">
         <origin xyz="0.020 0.115 0.155" rpy="0 0 ${pi}"/>
       </xacro:raspi_camera>
     </xacro:if>
     <xacro:if value="${raspicam_mount == 'downward'}">
-      <xacro:raspi_camera name="raspicam" connected_to="base_link">
+      <xacro:raspi_camera name="${tf_prefix}raspicam" connected_to="${tf_prefix}base_link">
         <origin xyz="0.1 0.090 0.145" rpy="3.14159 -1.25 0.0"/>
       </xacro:raspi_camera>
     </xacro:if>
     <xacro:if value="${raspicam_mount == 'ahead'}">
-      <xacro:raspi_camera name="raspicam" connected_to="base_link">
+      <xacro:raspi_camera name="${tf_prefix}raspicam" connected_to="${tf_prefix}base_link">
         <origin xyz="0.095 0.061 0.10" rpy="0 1.5707 0"/>
       </xacro:raspi_camera>

File: magni_description/urdf/sensors/raspi_camera.xacro (robot description, xacro)
@@ -1,5 +1,5 @@
 <?xml version="1.0" encoding="utf-8"?>
 <robot xmlns:xacro="http://wiki.ros.org/xacro">
-  <xacro:macro name="raspi_camera" params="name:='' connected_to:='' *origin">
+  <xacro:macro name="raspi_camera" params="name connected_to:='' *origin">
     <xacro:unless value="${connected_to == ''}">
       <joint name="${name}_joint" type="fixed">
